Commit message: Added instantiation of FT sensor joint and link macro

File: mymav_description/urdf/firefly.xacro (robot description, xacro)
@@ -59,6 +59,12 @@
     <xacro:insert_block name="body_inertia" />
   </xacro:multirotor_base_macro>
+<!--~~~~~~~~~~~~~~~~~~~~~~~~~~~~~~~~~~~~~-->
+  <!--Instantiate joints and link for FT sensor -->
+  <xacro:ft_joints_link
+    robot_namespace="${namespace}">
+  </xacro:ft_joints_link>
+<!--_______________________________________-->
   <!-- Instantiate rotors -->
-<xacro:vertical_rotor
+  <xacro:vertical_rotor
     robot_namespace="${namespace}"
     suffix="front_left"

File: mymav_description/urdf/multirotor_base.xacro (robot description, xacro)
@@ -73,4 +73,57 @@
     </gazebo>
   </xacro:macro>
+		<!--~~~~~~~~~~~~~~~~~~~~~~~~~~~~~~~~~~~~~~~~~~~~~~~~~~~~~~~~~~~~~-->
+    <!-- ATTACH MULTIROTOR_FT_PLUGIN TO THE BASE+_LINK -->
+  <xacro:macro name="ft_joints_link" params="robot_namespace">
+		<!--joint attached right to the base-->
+		<joint name="${robot_namespace}/ft_joint_start" type="fixed">
+			<origin xyz="0 0 0" rpy="0 0 0" />
+      <parent link="${robot_namespace}/base_link" />
+      <child link="${robot_namespace}/ft_link" />
+		</joint>
+		<!--extension to the ft sensor link-->
+		<link name="${robot_namespace}/ft_link">
+			<visual>
+        <geometry>
+           <box size="0.01 0.01 0.1"/>
+        </geometry>
+      </visual>
+      <collision>
+        <origin xyz="0 0 0" rpy="0 0 0"/>
+        <geometry>
+           <box size="0.01 0.01 0.1"/>
+        </geometry>
+      </collision>
+		</link>
+		<gazebo reference="${robot_namespace}/ft_link">
+      <material>Gazebo/White</material>
+    </gazebo>
+    <gazebo reference="${robot_namespace}/ft_joint_start">
+    	<provideFeedback>true</provideFeedback>
+		</gazebo>
+<!-- The ft_sensor plugin -->
+		<gazebo>
+    	<plugin name="ft_sensor" filename="libgazebo_ros_ft_sensor.so">
+        <updateRate>100.0</updateRate>
+        <topicName>ft_sensor_topic</topicName>
+        <jointName>firefly/ft_joint_start</jointName>
+    	</plugin>
+		</gazebo>
+    <!-- The ft_sensor plugin  -->
+    <!--gazebo>
+        <plugin name="ft_sensor" filename="libgazebo_ros_ft_sensor.so">
+          <updateRate>100.0</updateRate>
+          <robotNamespace>${robot_namespace}</robotNamespace>
+          <topicName>ft_sensor_topic</topicName>
+          <jointName>${robot_namespace}/ft_joint_finish</jointName>
+          <noise>
+            <type>gaussian</type>
+            <mean>0.0</mean>
+            <stddev>0.0001</stddev>
+        </noise>
+        </plugin>
+    </gazebo-->
+  </xacro:macro>
+<!--_______________________________________________________________-->
   <!-- Rotor joint and link -->
   <xacro:macro name="vertical_rotor"

Commit message: launch file changes, addition of a controller
Signed-off-by: BevandaFER <petar.bevanda@fer.hr>

File: mymav_description/urdf/firefly.xacro (robot description, xacro)
@@ -61,7 +61,12 @@
 <!--~~~~~~~~~~~~~~~~~~~~~~~~~~~~~~~~~~~~~-->
   <!--Instantiate joints and link for FT sensor -->
-  <xacro:ft_joints_link
-    robot_namespace="${namespace}">
-  </xacro:ft_joints_link>
+  <xacro:ft_senzor
+    robot_namespace="${namespace}"
+    masa="0.00001"
+		x="0.025"
+		y="0.025"
+		z="0.00005"
+>
+  </xacro:ft_senzor>
 <!--_______________________________________-->
   <!-- Instantiate rotors -->

File: mymav_description/urdf/multirotor_base.xacro (robot description, xacro)
@@ -64,4 +64,24 @@
       </collision>
     </link>
+		<!--joint attached right to the base>
+		<joint name="${robot_namespace}/ft_base_joint" type="fixed">
+			<origin xyz="0 0 -0.02" rpy="0 0 0" />
+      <parent link="${robot_namespace}/base_link" />
+      <child link="${robot_namespace}/ft_base_link" />
+		</joint-->
+		<!--extension to the ft sensor link>
+		<link name="${robot_namespace}/ft_base_link">
+			<visual>
+        <geometry>
+           <box size="0.01 0.01 0.1"/>
+        </geometry>
+      </visual>
+      <collision>
+        <origin xyz="0 0 0" rpy="0 0 0"/>
+        <geometry>
+           <box size="0.01 0.01 0.05"/>
+        </geometry>
+      </collision>
+		</link-->
     <!-- attach multirotor_base_plugin to the base_link -->
     <gazebo>
@@ -75,46 +95,51 @@
 		<!--~~~~~~~~~~~~~~~~~~~~~~~~~~~~~~~~~~~~~~~~~~~~~~~~~~~~~~~~~~~~~-->
     <!-- ATTACH MULTIROTOR_FT_PLUGIN TO THE BASE+_LINK -->
-  <xacro:macro name="ft_joints_link" params="robot_namespace">
-		<!--joint attached right to the base-->
-		<joint name="${robot_namespace}/ft_joint_start" type="fixed">
+  <xacro:macro name="ft_senzor" params="robot_namespace x y z masa">
+		<joint name="${robot_namespace}/ft_joint" type="revolute">
 			<origin xyz="0 0 0" rpy="0 0 0" />
       <parent link="${robot_namespace}/base_link" />
-      <child link="${robot_namespace}/ft_link" />
+      <child link="${robot_namespace}/ft_contact_link" />
+			<limit effort="30" velocity="1.0" lower="0" upper="0" />
 		</joint>
-		<!--extension to the ft sensor link-->
-		<link name="${robot_namespace}/ft_link">
+		<link name="${robot_namespace}/ft_contact_link">
 			<visual>
-        <geometry>
+			<origin xyz="0 0 -0.05" rpy="0 0 0" />
+        <geometry>`
            <box size="0.01 0.01 0.1"/>
         </geometry>
       </visual>
       <collision>
-        <origin xyz="0 0 0" rpy="0 0 0"/>
+        <origin xyz="0 0 -0.05" rpy="0 0 0" />
         <geometry>
            <box size="0.01 0.01 0.1"/>
         </geometry>
       </collision>
+			<inertial>
+			<origin xyz="0 0 -0.05" rpy="0 0 0" />
+        <mass value="0.00001" />
+        <xacro:box_inertia x="${x}" y="${y}" z="${z}" mass="${mass}" />
+      </inertial>
 		</link>
-		<gazebo reference="${robot_namespace}/ft_link">
+		<!--gazebo reference="${robot_namespace}/ft_link">
       <material>Gazebo/White</material>
-    </gazebo>
-    <gazebo reference="${robot_namespace}/ft_joint_start">
+    </gazebo-->
+    <!--gazebo reference="${robot_namespace}/ft_joint_start">
     	<provideFeedback>true</provideFeedback>
-		</gazebo>
+		</gazebo-->
 <!-- The ft_sensor plugin -->
-		<gazebo>
+		<!--gazebo>
     	<plugin name="ft_sensor" filename="libgazebo_ros_ft_sensor.so">
         <updateRate>100.0</updateRate>
         <topicName>ft_sensor_topic</topicName>
-        <jointName>firefly/ft_joint_start</jointName>
+        <jointName>${robot_namespace}/ft_joint_start</jointName>
     	</plugin>
-		</gazebo>
+		</gazebo>-->
     <!-- The ft_sensor plugin  -->
-    <!--gazebo>
+    <gazebo>
         <plugin name="ft_sensor" filename="libgazebo_ros_ft_sensor.so">
           <updateRate>100.0</updateRate>
           <robotNamespace>${robot_namespace}</robotNamespace>
           <topicName>ft_sensor_topic</topicName>
-          <jointName>${robot_namespace}/ft_joint_finish</jointName>
+          <jointName>${robot_namespace}/ft_joint</jointName>
           <noise>
             <type>gaussian</type>
@@ -123,5 +148,5 @@
         </noise>
         </plugin>
-    </gazebo-->
+    </gazebo>
   </xacro:macro>
 <!--_______________________________________________________________-->
