Commit message: mymav_description file structure overhaul; added <provideFeedback> tag to ensure that the ft sensor functions properly

File: mymav_description/urdf/component_snippets.xacro (robot description, xacro)
@@ -834,4 +834,3 @@
     </xacro:mavlink_interface_macro>
   </xacro:macro>
-		<!-- F/T Sensor -->
 </robot>

File: mymav_description/urdf/firefly.urdf.xacro (robot description, xacro)
@@ -21,5 +21,5 @@
   <xacro:property name="rotor_velocity_slowdown_sim" value="10" />
   <xacro:property name="use_mesh_file" value="true" />
-  <xacro:property name="mesh_file" value="package://rotors_description/meshes/firefly.dae" />
+  <xacro:property name="mesh_file" value="package://mymav_description/meshes/firefly.dae" />
   <xacro:property name="mass" value="1.5" /> <!-- [kg] -->
   <xacro:property name="body_width" value="0.1" /> <!-- [m] -->
@@ -47,5 +47,5 @@
   </xacro:property>
   <!-- Included URDF Files -->
-  <xacro:include filename="$(find rotors_description)/urdf/multirotor_base.xacro" />
+  <xacro:include filename="$(find mymav_description)/urdf/multirotor_base.urdf.xacro" />
   <!-- Instantiate multirotor_base_macro once -->
   <xacro:multirotor_base_macro
@@ -61,5 +61,5 @@
 <!--~~~~~~~~~~~~~~~~~~~~~~~~~~~~~~~~~~~~~-->
   <!--Instantiate joints and link for FT sensor -->
-  <xacro:ft_senzor
+  <xacro:ft_sensor
     robot_namespace="${namespace}"
     masa="0.00001"
@@ -67,8 +67,8 @@
 		y="0.025"
 		z="0.00005"
->
-  </xacro:ft_senzor>
+    >
+  </xacro:ft_sensor>
 <!--_______________________________________-->
-  <!-- Instantiate rotors -->
+  <!-- Instantiate mymav -->
   <xacro:vertical_rotor
     robot_namespace="${namespace}"

File: mymav_description/urdf/multirotor_base.urdf.xacro (robot description, xacro)
@@ -64,24 +64,4 @@
       </collision>
     </link>
-		<!--joint attached right to the base>
-		<joint name="${robot_namespace}/ft_base_joint" type="fixed">
-			<origin xyz="0 0 -0.02" rpy="0 0 0" />
-      <parent link="${robot_namespace}/base_link" />
-      <child link="${robot_namespace}/ft_base_link" />
-		</joint-->
-		<!--extension to the ft sensor link>
-		<link name="${robot_namespace}/ft_base_link">
-			<visual>
-        <geometry>
-           <box size="0.01 0.01 0.1"/>
-        </geometry>
-      </visual>
-      <collision>
-        <origin xyz="0 0 0" rpy="0 0 0"/>
-        <geometry>
-           <box size="0.01 0.01 0.05"/>
-        </geometry>
-      </collision>
-		</link-->
     <!-- attach multirotor_base_plugin to the base_link -->
     <gazebo>
@@ -93,62 +73,5 @@
     </gazebo>
   </xacro:macro>
-		<!--~~~~~~~~~~~~~~~~~~~~~~~~~~~~~~~~~~~~~~~~~~~~~~~~~~~~~~~~~~~~~-->
-    <!-- ATTACH MULTIROTOR_FT_PLUGIN TO THE BASE+_LINK -->
-  <xacro:macro name="ft_senzor" params="robot_namespace x y z masa">
-		<joint name="${robot_namespace}/ft_joint" type="revolute">
-			<origin xyz="0 0 0" rpy="0 0 0" />
-      <parent link="${robot_namespace}/base_link" />
-      <child link="${robot_namespace}/ft_contact_link" />
-			<limit effort="30" velocity="1.0" lower="0" upper="0" />
-		</joint>
-		<link name="${robot_namespace}/ft_contact_link">
-			<visual>
-			<origin xyz="0 0 -0.05" rpy="0 0 0" />
-        <geometry>`
-           <box size="0.01 0.01 0.1"/>
-        </geometry>
-      </visual>
-      <collision>
-        <origin xyz="0 0 -0.05" rpy="0 0 0" />
-        <geometry>
-           <box size="0.01 0.01 0.1"/>
-        </geometry>
-      </collision>
-			<inertial>
-			<origin xyz="0 0 -0.05" rpy="0 0 0" />
-        <mass value="0.00001" />
-        <xacro:box_inertia x="${x}" y="${y}" z="${z}" mass="${mass}" />
-      </inertial>
-		</link>
-		<!--gazebo reference="${robot_namespace}/ft_link">
-      <material>Gazebo/White</material>
-    </gazebo-->
-    <!--gazebo reference="${robot_namespace}/ft_joint_start">
-    	<provideFeedback>true</provideFeedback>
-		</gazebo-->
-<!-- The ft_sensor plugin -->
-		<!--gazebo>
-    	<plugin name="ft_sensor" filename="libgazebo_ros_ft_sensor.so">
-        <updateRate>100.0</updateRate>
-        <topicName>ft_sensor_topic</topicName>
-        <jointName>${robot_namespace}/ft_joint_start</jointName>
-    	</plugin>
-		</gazebo>-->
-    <!-- The ft_sensor plugin  -->
-    <gazebo>
-        <plugin name="ft_sensor" filename="libgazebo_ros_ft_sensor.so">
-          <updateRate>100.0</updateRate>
-          <robotNamespace>${robot_namespace}</robotNamespace>
-          <topicName>ft_sensor_topic</topicName>
-          <jointName>${robot_namespace}/ft_joint</jointName>
-          <noise>
-            <type>gaussian</type>
-            <mean>0.0</mean>
-            <stddev>0.0001</stddev>
-        </noise>
-        </plugin>
-    </gazebo>
-  </xacro:macro>
-<!--_______________________________________________________________-->
+-->
   <!-- Rotor joint and link -->
   <xacro:macro name="vertical_rotor"
@@ -175,5 +98,5 @@
           </xacro:if>
           <xacro:unless value="${use_own_mesh}">
-            <mesh filename="package://rotors_description/meshes/propeller_${direction}.dae"
+            <mesh filename="package://mymav_description/meshes/propeller_${direction}.dae"
               scale="${radius_rotor} ${radius_rotor} ${radius_rotor}" /> <!-- The propeller meshes have a radius of 1m -->
             <!-- <box size="${2*radius_rotor} 0.01 0.005"/> -->
