Commit message: Added Kp and Kd parameters for modeling force sensor

File: mymav_description/urdf/firefly.gazebo.xacro (robot description, xacro)
@@ -42,9 +42,11 @@
     <!-- ATTACH MULTIROTOR_FT_PLUGIN TO THE BASE+_LINK -->
   <xacro:macro name="ft_sensor" params="robot_namespace x y z masa">
-    <joint name="${namespace}/ft_joint" type="revolute">
+    <joint name="${namespace}/ft_joint" type="prismatic">
       <origin xyz="0 0 0" rpy="0 0 0" />
       <parent link="${namespace}/base_link" />
       <child link="${namespace}/ft_contact_link" />
       <limit effort="0" velocity="0" lower="0" upper="0" />
+      <axis xyz="0 0 1"/>
+      <!--dynamics spring_stiffness='1000000' spring_reference='0' damping='0' friction='0'/-->
     </joint>
     <link name="${namespace}/ft_contact_link">
@@ -67,4 +69,9 @@
       </inertial>
     </link>
+    <gazebo reference="${robot_namespace}/ft_contact_link">
+      <provideFeedback>True</provideFeedback>
+      <kp>6000</kp>
+      <kd>60000</kd>
+    </gazebo>
     <gazebo reference="${namespace}/ft_joint">
       <provideFeedback>true</provideFeedback>

Commit message: Added new launch files; Changed world file to suit sim requirements; Added joy control; Tuned FT sensor contact response

File: mymav_description/urdf/firefly.gazebo.xacro (robot description, xacro)
@@ -41,29 +41,29 @@
     <!--~~~~~~~~~~~~~~~~~~~~~~~~~~~~~~~~~~~~~~~~~~~~~~~~~~~~~~~~~~~~~-->
     <!-- ATTACH MULTIROTOR_FT_PLUGIN TO THE BASE+_LINK -->
-  <xacro:macro name="ft_sensor" params="robot_namespace x y z masa">
-    <joint name="${namespace}/ft_joint" type="prismatic">
+  <xacro:macro name="ft_sensor" params="robot_namespace x y z mass">
+    <joint name="${robot_namespace}/ft_joint" type="prismatic">
       <origin xyz="0 0 0" rpy="0 0 0" />
-      <parent link="${namespace}/base_link" />
-      <child link="${namespace}/ft_contact_link" />
+      <parent link="${robot_namespace}/base_link" />
+      <child link="${robot_namespace}/ft_contact_link" />
       <limit effort="0" velocity="0" lower="0" upper="0" />
       <axis xyz="0 0 1"/>
       <!--dynamics spring_stiffness='1000000' spring_reference='0' damping='0' friction='0'/-->
     </joint>
-    <link name="${namespace}/ft_contact_link">
+    <link name="${robot_namespace}/ft_contact_link">
       <visual>
-      <origin xyz="0 0 -0.05" rpy="0 0 0" />
+      <origin xyz="0 0 -${z/2}" rpy="0 0 0" />
         <geometry>`
-           <box size="0.01 0.01 0.1"/>
+           <box size="${x} ${y} ${z}"/>
         </geometry>
       </visual>
       <collision>
-        <origin xyz="0 0 -0.05" rpy="0 0 0" />
+        <origin xyz="0 0 -${z/2}" rpy="0 0 0" />
         <geometry>
-           <box size="0.01 0.01 0.1"/>
+           <box size="${x} ${y} ${z}" />
         </geometry>
       </collision>
       <inertial>
-      <origin xyz="0 0 -0.05" rpy="0 0 0" />
-        <mass value="0.00001" />
+      <origin xyz="0 0 -${z/2}" rpy="0 0 0" />
+        <mass value="${mass}" />
         <xacro:box_inertia x="${x}" y="${y}" z="${z}" mass="${mass}" />
       </inertial>
@@ -71,14 +71,15 @@
     <gazebo reference="${robot_namespace}/ft_contact_link">
       <provideFeedback>True</provideFeedback>
-      <kp>6000</kp>
-      <kd>60000</kd>
+      <kp>1.0e+9</kp>
+      <kd>5.0e+5</kd>
     </gazebo>
-    <gazebo reference="${namespace}/ft_joint">
+    <gazebo reference="${robot_namespace}/ft_joint">
       <provideFeedback>true</provideFeedback>
     </gazebo>
-    <gazebo reference="${namespace}/ft_contact_link">
+    <gazebo reference="${robot_namespace}/ft_contact_link">
       <provideFeedback>true</provideFeedback>
+      <material>Gazebo/Orange</material>
     </gazebo>
-    <gazebo reference="${namespace}/base_link">
+    <gazebo reference="${robot_namespace}/base_link">
       <provideFeedback>true</provideFeedback>
     </gazebo>
@@ -87,7 +88,7 @@
         <plugin name="ft_sensor" filename="libgazebo_ros_ft_sensor.so">
           <updateRate>100.0</updateRate>
-          <robotNamespace>${namespace}</robotNamespace>
+          <robotNamespace>${robot_namespace}</robotNamespace>
           <topicName>ft_sensor_topic</topicName>
-          <jointName>${namespace}/ft_joint</jointName>
+          <jointName>${robot_namespace}/ft_joint</jointName>
           <noise>
             <type>gaussian</type>

File: mymav_description/urdf/firefly.urdf.xacro (robot description, xacro)
@@ -1,19 +1,3 @@
 <?xml version="1.0"?>
-<!--
-  Copyright 2015 Fadri Furrer, ASL, ETH Zurich, Switzerland
-  Copyright 2015 Michael Burri, ASL, ETH Zurich, Switzerland
-  Copyright 2015 Mina Kamel, ASL, ETH Zurich, Switzerland
-  Copyright 2015 Janosch Nikolic, ASL, ETH Zurich, Switzerland
-  Copyright 2015 Markus Achtelik, ASL, ETH Zurich, Switzerland
-  Licensed under the Apache License, Version 2.0 (the "License");
-  you may not use this file except in compliance with the License.
-  You may obtain a copy of the License at
-  http://www.apache.org/licenses/LICENSE-2.0
-  Unless required by applicable law or agreed to in writing, software
-  distributed under the License is distributed on an "AS IS" BASIS,
-  WITHOUT WARRANTIES OR CONDITIONS OF ANY KIND, either express or implied.
-  See the License for the specific language governing permissions and
-  limitations under the License.
--->
 <robot name="firefly" xmlns:xacro="http://ros.org/wiki/xacro">
   <!-- Properties -->
@@ -63,8 +47,8 @@
   <xacro:ft_sensor
     robot_namespace="${namespace}"
-    masa="0.00001"
-		x="0.025"
-		y="0.025"
-		z="0.00005"
+    mass="0.001"
+    x="0.01"
+    y="0.01"
+    z="0.1"
     >
   </xacro:ft_sensor>

File: mymav_description/urdf/multirotor_base.urdf.xacro (robot description, xacro)
@@ -133,3 +133,57 @@
     </gazebo>
   </xacro:macro>
+<!-- Macro to add a generic odometry sensor. -->
+  <xacro:macro name="odometry_plugin_macro"
+    params="
+      namespace odometry_sensor_suffix parent_link pose_topic pose_with_covariance_topic
+      position_topic transform_topic odometry_topic parent_frame_id child_frame_id
+      mass_odometry_sensor measurement_divisor measurement_delay unknown_delay
+      noise_normal_position noise_normal_quaternion noise_normal_linear_velocity
+      noise_normal_angular_velocity noise_uniform_position
+      noise_uniform_quaternion noise_uniform_linear_velocity
+      noise_uniform_angular_velocity enable_odometry_map odometry_map
+      image_scale *inertia *origin">
+    <!-- odometry link -->
+    <link name="${namespace}/odometry_sensor${odometry_sensor_suffix}_link">
+      <inertial>
+        <xacro:insert_block name="inertia" />
+        <mass value="${mass_odometry_sensor}" />  <!-- [kg] -->
+      </inertial>
+    </link>
+    <!-- odometry joint -->
+    <joint name="${namespace}/odometry_sensor${odometry_sensor_suffix}_joint" type="revolute">
+      <parent link="${parent_link}" />
+      <xacro:insert_block name="origin" />
+      <child link="${namespace}/odometry_sensor${odometry_sensor_suffix}_link" />
+      <limit upper="0" lower="0" effort="0" velocity="0" />
+    </joint>
+    <gazebo>
+      <plugin filename="librotors_gazebo_odometry_plugin.so" name="odometry_sensor${odometry_sensor_suffix}">
+        <linkName>${namespace}/odometry_sensor${odometry_sensor_suffix}_link</linkName>
+        <robotNamespace>${namespace}</robotNamespace>
+        <poseTopic>${pose_topic}</poseTopic>
+        <poseWithCovarianceTopic>${pose_with_covariance_topic}</poseWithCovarianceTopic>
+        <positionTopic>${position_topic}</positionTopic>
+        <transformTopic>${transform_topic}</transformTopic>
+        <odometryTopic>${odometry_topic}</odometryTopic>
+        <parentFrameId>${parent_frame_id}</parentFrameId> <!-- Use the scoped link name here. e.g. Model::link. -->
+        <childFrameId>${child_frame_id}</childFrameId>
+        <measurementDivisor>${measurement_divisor}</measurementDivisor> <!-- only every (seq % measurementDivisor) == 0 measurement is published [int] -->
+        <measurementDelay>${measurement_delay}</measurementDelay> <!-- time that measurement gets held back before it's published in [simulation cycles (int)] -->
+        <unknownDelay>${unknown_delay}</unknownDelay> <!-- additional delay, that just gets added to the timestamp [s] -->
+        <noiseNormalPosition>${noise_normal_position}</noiseNormalPosition> <!-- standard deviation of additive white gaussian noise [m] -->
+        <noiseNormalQuaternion>${noise_normal_quaternion}</noiseNormalQuaternion> <!-- standard deviation white gaussian noise [rad]: q_m = q*quaternionFromSmallAngleApproximation(noiseNormalQ) -->
+        <noiseNormalLinearVelocity>${noise_normal_linear_velocity}</noiseNormalLinearVelocity> <!-- standard deviation of additive white gaussian noise [m/s] -->
+        <noiseNormalAngularVelocity>${noise_normal_angular_velocity}</noiseNormalAngularVelocity> <!-- standard deviation of additive white gaussian noise [rad/s] -->
+        <noiseUniformPosition>${noise_uniform_position}</noiseUniformPosition> <!-- symmetric bounds of uniform noise [m] -->
+        <noiseUniformQuaternion>${noise_uniform_quaternion}</noiseUniformQuaternion> <!-- symmetric bounds of uniform noise [rad], computation see above -->
+        <noiseUniformLinearVelocity>${noise_uniform_linear_velocity}</noiseUniformLinearVelocity> <!-- symmetric bounds of uniform noise [m/s] -->
+        <noiseUniformAngularVelocity>${noise_uniform_angular_velocity}</noiseUniformAngularVelocity> <!-- symmetric bounds of uniform noise [rad/s] -->
+        <xacro:if value="${enable_odometry_map}">
+          <covarianceImage>package://rotors_gazebo/resource/${odometry_map}</covarianceImage> <!-- a bitmap image describing where the sensor works (white), and where not (black) -->
+          <covarianceImageScale>${image_scale}</covarianceImageScale> <!-- the scale of the image in the gazebo world, if set to 1.0, 1 pixel in the image corresponds to 1 meter in the world -->
+        </xacro:if>
+      </plugin>
+    </gazebo>
+  </xacro:macro>
 </robot>

Commit message: tuned stuff for FT sensor readings

File: mymav_description/urdf/firefly.gazebo.xacro (robot description, xacro)
@@ -1,19 +1,3 @@
 <?xml version="1.0"?>
-<!--
-  Copyright 2015 Fadri Furrer, ASL, ETH Zurich, Switzerland
-  Copyright 2015 Michael Burri, ASL, ETH Zurich, Switzerland
-  Copyright 2015 Mina Kamel, ASL, ETH Zurich, Switzerland
-  Copyright 2015 Janosch Nikolic, ASL, ETH Zurich, Switzerland
-  Copyright 2015 Markus Achtelik, ASL, ETH Zurich, Switzerland
-  Licensed under the Apache License, Version 2.0 (the "License");
-  you may not use this file except in compliance with the License.
-  You may obtain a copy of the License at
-  http://www.apache.org/licenses/LICENSE-2.0
-  Unless required by applicable law or agreed to in writing, software
-  distributed under the License is distributed on an "AS IS" BASIS,
-  WITHOUT WARRANTIES OR CONDITIONS OF ANY KIND, either express or implied.
-  See the License for the specific language governing permissions and
-  limitations under the License.
--->
 <robot name="firefly" xmlns:xacro="http://ros.org/wiki/xacro">
   <xacro:include filename="$(find mymav_description)/urdf/component_snippets.xacro" />
@@ -48,9 +32,9 @@
       <limit effort="0" velocity="0" lower="0" upper="0" />
       <axis xyz="0 0 1"/>
-      <!--dynamics spring_stiffness='1000000' spring_reference='0' damping='0' friction='0'/-->
+      <!--dynamics spring_stiffness='1000000' spring_reference='0' damping='0.7' friction='0'/-->
     </joint>
     <link name="${robot_namespace}/ft_contact_link">
       <visual>
-      <origin xyz="0 0 -${z/2}" rpy="0 0 0" />
+      <origin xyz="0 0 ${-z/2}" rpy="0 0 0" />
         <geometry>`
            <box size="${x} ${y} ${z}"/>
@@ -58,5 +42,5 @@
       </visual>
       <collision>
-        <origin xyz="0 0 -${z/2}" rpy="0 0 0" />
+        <origin xyz="0 0 ${-z/2}" rpy="0 0 0" />
         <geometry>
            <box size="${x} ${y} ${z}" />
@@ -64,14 +48,9 @@
       </collision>
       <inertial>
-      <origin xyz="0 0 -${z/2}" rpy="0 0 0" />
+      <origin xyz="0 0 ${-z/2}" rpy="0 0 0" />
         <mass value="${mass}" />
         <xacro:box_inertia x="${x}" y="${y}" z="${z}" mass="${mass}" />
       </inertial>
     </link>
-    <gazebo reference="${robot_namespace}/ft_contact_link">
-      <provideFeedback>True</provideFeedback>
-      <kp>1.0e+9</kp>
-      <kd>5.0e+5</kd>
-    </gazebo>
     <gazebo reference="${robot_namespace}/ft_joint">
       <provideFeedback>true</provideFeedback>
@@ -79,4 +58,6 @@
     <gazebo reference="${robot_namespace}/ft_contact_link">
       <provideFeedback>true</provideFeedback>
+      <kp>1.0e+9</kp>
+      <kd>5.0e+5</kd>
       <material>Gazebo/Orange</material>
     </gazebo>

File: mymav_description/urdf/firefly.urdf.xacro (robot description, xacro)
@@ -4,5 +4,5 @@
   <xacro:property name="namespace" value="$(arg namespace)" />
   <xacro:property name="rotor_velocity_slowdown_sim" value="10" />
-  <xacro:property name="use_mesh_file" value="true" />
+  <xacro:property name="use_mesh_file" value="false" />
   <xacro:property name="mesh_file" value="package://mymav_description/meshes/firefly.dae" />
   <xacro:property name="mass" value="1.5" /> <!-- [kg] -->
